File: kicad/k1-aioc/k1-aioc.kicad_sch (KiCad schematic)
At the start: 46 parts, among them J1 12401832E402A, J2 Conn_01x07_Male, Q1 BC847BS, U1 MIC5330-SSYML, U2 STM32F373CBTx, Y1 8MHz/20pF

Commit message: Added A new Connector
Added a new connector.
Parts:
- USB1: renamed from J1; value 12401832E402A -> HX TYPE-C 24P QCHT; footprint AIOC:USB_C_Receptacle_Amphenol_12401832E40-2A -> C5178545:TYPE-C-SMD_TYPE-C-24P-QCHT; symbol Connector:USB_C_Receptacle_USB2.0 -> C5178545:HXTYPE-C24PQCHT; LCSC C464604 -> (none); LCSC Part (none) -> C5178545
Connections:
- net GND: no longer USB1.A1 (GND), USB1.A12 (GND), USB1.B1 (GND), USB1.B12 (GND), USB1.S1 (SHIELD)
- net USB-DN: now also USB1.B5 (CC2), USB1.B6 (DP2); no longer USB1.A7 (D-), USB1.B7 (D-)
- net USB-DP: now also USB1.B3 (SSIXn2), USB1.B4 (VBUS); no longer USB1.A6 (D+), USB1.B6 (D+)
- net VBUS: now also USB1.B11 (SSRXp1); no longer USB1.A4 (VBUS), USB1.A9 (VBUS), USB1.B4 (VBUS), USB1.B9 (VBUS)
- net at R6.2: now also USB1.B8 (SUB2); no longer USB1.B5 (CC2)
- net at R7.2: now also USB1.B9 (VBUS); no longer USB1.A5 (CC1)

Commit message: End of day progress
End of day progress
Parts:
- renumbered USB1 to J1
Connections:
- net GND: now also J1.25, J1.A1 (GND), J1.A12 (GND), J1.B1 (GND), J1.B12 (GND), R7.2; no longer R7.1
- net USB-DN: now also J1.A7 (DN2), J1.B7 (DN2); no longer J1.B5 (CC2), J1.B6 (DP2)
- net USB-DP: now also J1.A6 (DP1), J1.B6 (DP2); no longer J1.B3 (SSIXn2), J1.B4 (VBUS)
- net VBUS: now also FB2.1, J1.A4 (VBUS), J1.A9 (VBUS), J1.B4 (VBUS), J1.B9 (VBUS); no longer FB2.2, J1.B11 (SSRXp1)
- net VIN: now also FB2.2; no longer FB2.1
- net at R6.2: now also J1.B5 (CC2); no longer J1.B8 (SUB2)
- net at J1.A5 (CC1): now also R7.1
Other:
- note added: "MIC5330: dual low-dropout (LDO) linear regulator"
- moved on the sheet: C3, C4, C5, C6, FB1, FB2, J1, R1, R6, R7, U1
