File: kicad/k1-aioc/k1-aioc.kicad_sch (KiCad schematic)
At the start: 46 parts, among them J1 HX TYPE-C 24P QCHT, J2 Conn_01x07_Male, Q1 BC847BS, U1 MIC5330-SSYML-TR, U2 STM32F302CBT6, Y1 8MHz/20pF

Commit message: Getting order ready for testing
Getting order ready for testing.
Parts:
- D2: value RED -> LED; footprint LED_SMD:LED_0603_1608Metric -> (none); LCSC C2286 -> (none)
- D3, D4: value N.M. -> LED; footprint LED_SMD:LED_0603_1608Metric -> (none)
- LED1: renamed from D1; value GREEN -> XL-1608UGC-04; footprint LED_SMD:LED_0603_1608Metric -> C965804:LED0603-RD_GREEN; symbol Device:LED -> C965804:XL-1608UGC-04; LCSC C72043 -> (none); LCSC Part (none) -> C965804
Connections:
- net +3V3: now also U1.8 (VOUT1)
- net GND: now also U1.2 (GND), U1.9 (EP)
- net VIN: now also U1.1 (VIN), U1.4 (EN2), U1.5 (EN1)
- net at D2.2 (A), D3.1 (K), D4.2 (A)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: no longer LED1.1 (K)
- net at D2.1 (K), D3.2 (A), D4.1 (K)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: no longer LED1.2 (A)
- net at C5.1, FB1.2: now also U1.7 (VOUT2)
- net at U1.3 (BYP): now also C3.1
Other:
- moved on the sheet: C3, C4, C5, C6, FB1, FB2, U1
