File: kicad/k1-aioc/k1-aioc.kicad_pcb (KiCad board)
At the start: 2 copper layers, 21 x 31.5 mm, 47 parts, among them J1 12401832E402A, J2 Conn_01x07_Male, Q1 BC847BS, U1 MIC5330-SSYML, U2 STM32F373CBTx, Y1 8MHz/20pF

Commit message: tweaks
Tweaks and changes.
Parts:
- J1: value 12401832E402A -> HX TYPE-C 24P QCHT; footprint AIOC:USB_C_Receptacle_Amphenol_12401832E40-2A -> C5178545:TYPE-C-SMD_TYPE-C-24P-QCHT
- U1: value MIC5330-SSYML -> MIC5330-SSYML-TR; footprint AIOC:Micrel_MLF-8-1EP_2x2mm_P0.5mm_EP0.6x1.2mm -> C144168:MLF-8_L2.0-W2.0-P0.50-BL-EP
- U2: value STM32F373CBTx -> STM32F302CBT6
- turned U1 to 180 degrees
Connections:
- FB2 pad 1: /VIN -> /VBUS
- FB2 pad 2: /VBUS -> /VIN
- J1 pad A10: (no net) -> unconnected-(J1-SSRXn2-PadA10)
- J1 pad A11: (no net) -> unconnected-(J1-SSRXp2-PadA11)
- J1 pad A2: (no net) -> unconnected-(J1-SSTXp1-PadA2)
- J1 pad A3: (no net) -> unconnected-(J1-SSTXn1-PadA3)
- J1 pad A5: Net-(J1-PadA5) -> Net-(J1-CC1)
- J1 pad B10: (no net) -> unconnected-(J1-SSRXn1-PadB10)
- J1 pad B11: (no net) -> unconnected-(J1-SSRXp1-PadB11)
- J1 pad B2: (no net) -> unconnected-(J1-SSTXp2-PadB2)
- J1 pad B3: (no net) -> unconnected-(J1-SSIXn2-PadB3)
- R7 pad 1: GND -> Net-(J1-CC1)
- R7 pad 2: Net-(J1-PadA5) -> GND
- U1 pad 6: (no net) -> unconnected-(U1-NC-Pad6)
Routing:
- net (no net): track 0.00 -> 19.0 mm
- net Net-(J1-PadA5): track 10.1 -> 0.00 mm, vias 2 -> 0
- net Net-(J1-CC2): track 8.97 -> 0.00 mm
- net GND: vias 62 -> 64
Other:
- board text added: "dev-0.1"

Commit message: added my branch tag
added by github username and branch development tag to differentiate this board and it's changes from the origional.
Other:
- board text added: "cjemorton dev-0.1"
- board text removed: "dev-0.1"
Changed lines of the file:
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@@
 		)
 	)
-	(gr_text "dev-0.1"
-		(at 115 95.5 0)
+	(gr_text "cjemorton\ndev-0.1"
+		(at 116.5 105.5 0)
 		(layer "B.SilkS")
 		(effects
