File: kicad/k1-aioc/k1-aioc-dev-0.1.kicad_sch (KiCad schematic)
At the start: 46 parts, among them J1 HX TYPE-C 24P QCHT, J2 Conn_01x07_Male, Q1 BC847BS, U1 MIC5330-SSYML-TR, U2 STM32F302CBT6, Y1 8MHz/20pF

Commit message: Getting order ready for testing
Getting order ready for testing.
Parts:
- D2: value RED -> LED; footprint LED_SMD:LED_0603_1608Metric -> (none); LCSC C2286 -> (none)
- D3, D4: value N.M. -> LED; footprint LED_SMD:LED_0603_1608Metric -> (none)
- LED1: renamed from D1; value GREEN -> XL-1608UGC-04; footprint LED_SMD:LED_0603_1608Metric -> C965804:LED0603-RD_GREEN; symbol Device:LED -> C965804:XL-1608UGC-04; LCSC C72043 -> (none); LCSC Part (none) -> C965804
Connections:
- net at D2.2 (A), D3.1 (K), D4.2 (A)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: no longer LED1.1 (K)
- net at D2.1 (K), D3.2 (A), D4.1 (K)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: no longer LED1.2 (A)
Changed lines of the file:
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@@
 		(dnp no)
 		(property "Reference" "D3"
-			(at 170.18 143.51 0)
+			(at 166.37 144.78 0)
 			(effects
 				(font
@@
 			)
 		)
-		(property "Value" "N.M."
-			(at 170.18 146.05 0)
+		(property "Value" "LED"
+			(at 166.37 149.86 0)
 			(effects
 				(font
@@
 			)
 		)
-		(property "Footprint" "LED_SMD:LED_0603_1608Metric"
+		(property "Footprint" ""
 			(at 166.37 147.32 0)
 			(effects
@@
 			)
 		)
-		(property "Description" ""
+		(property "Description" "Light emitting diode"
 			(at 166.37 147.32 0)
 			(effects
@@
 					(size 1.27 1.27)
 				)
+				(hide yes)
 			)
 		)
-		(property "LCSC" ""
-			(at 164.7825 140.97 0)
+		(property "Sim.Pins" "1=K 2=A"
+			(at 166.37 147.32 0)
 			(effects
 				(font
@@
 	)
 	(symbol
-		(lib_id "Device:LED")
+		(lib_id "C965804:XL-1608UGC-04")
 		(at 158.75 152.4 0)
 		(unit 1)
@@
 		(dnp no)
 		(fields_autoplaced yes)
-		(property "Reference" "D1"
-			(at 157.1625 146.05 0)
+		(property "Reference" "LED1"
+			(at 157.99 143.51 0)
 			(effects
 				(font
@@
 			)
 		)
-		(property "Value" "GREEN"
-			(at 157.1625 148.59 0)
+		(property "Value" "XL-1608UGC-04"
+			(at 157.99 146.05 0)
 			(effects
 				(font
@@
 			)
 		)
-		(property "Footprint" "LED_SMD:LED_0603_1608Metric"
-			(at 158.75 152.4 0)
+		(property "Footprint" "C965804:LED0603-RD_GREEN"
+			(at 158.75 160.02 0)
 			(effects
 				(font
@@
 			)
 		)
-		(property "Datasheet" "~"
+		(property "Datasheet" ""
 			(at 158.75 152.4 0)
 			(effects
@@
 					(size 1.27 1.27)
 				)
+				(hide yes)
 			)
 		)
-		(property "LCSC" "C72043"
-			(at 157.1625 146.05 0)
+		(property "LCSC Part" "C965804"
+			(at 158.75 162.56 0)
 			(effects
 				(font
@@
 			(project ""
 				(path "/6b10ea87-c95d-4ec7-ad2b-5b0dcbbb7b7c"
-					(reference "D1")
+					(reference "LED1")
 					(unit 1)
 				)
@@
 			)
 		)
-		(property "Value" "N.M."
+		(property "Value" "LED"
 			(at 167.9575 161.29 0)
 			(effects
@@
 			)
 		)
-		(property "Footprint" "LED_SMD:LED_0603_1608Metric"
+		(property "Footprint" ""
 			(at 166.37 166.37 0)
 			(effects
@@
 			)
 		)
-		(property "Description" ""
+		(property "Description" "Light emitting diode"
 			(at 166.37 166.37 0)
 			(effects
@@
 					(size 1.27 1.27)
 				)
+				(hide yes)
 			)
 		)
-		(property "LCSC" ""
-			(at 167.9575 172.72 0)
+		(property "Sim.Pins" "1=K 2=A"
+			(at 166.37 166.37 0)
 			(effects
 				(font
@@
 			)
 		)
-		(property "Value" "RED"
+		(property "Value" "LED"
 			(at 160.3375 157.48 0)
 			(effects
@@
 			)
 		)
-		(property "Footprint" "LED_SMD:LED_0603_1608Metric"
+		(property "Footprint" ""
 			(at 158.75 162.56 0)
 			(effects
@@
 			)
 		)
-		(property "Description" ""
+		(property "Description" "Light emitting diode"
 			(at 158.75 162.56 0)
 			(effects
@@
 					(size 1.27 1.27)
 				)
+				(hide yes)
 			)
 		)
-		(property "LCSC" "C2286"
-			(at 160.3375 154.94 0)
+		(property "Sim.Pins" "1=K 2=A"
+			(at 158.75 162.56 0)
 			(effects
 				(font
